File: kicad-projects/MS20-VCF-Module/MS20-VCF-Module.kicad_sch (KiCad schematic)
At the start: 53 parts

Commit message: Finalized the VCF schematics
Parts:
- removed Q? (x2): Q_PNP_CBE, symbol Device:Q_PNP_CBE
- added Q1, Q2: 2N5401, symbol Device:Q_PNP_EBC
- added SW1: LP/BP/HP, symbol Switch:SW_DP3T
- C11, C12: renamed from C?; value C_Polarized -> 47uF
- D1, D2: renamed from D?; value LED -> GREEN
- J7: renamed from J?; value Conn_02x05_Odd_Even -> Power_EUR
- gave numbers to parts that had none: 42
Connections:
- net +12V: now also J7.10 (Pin_10), J7.9 (Pin_9); no longer J7.1 (Pin_1), J7.2 (Pin_2)
- net -12V: now also J7.1 (Pin_1), J7.2 (Pin_2); no longer J7.10 (Pin_10), J7.9 (Pin_9)
- net GND: now also Q2.2 (B), SW1.5; no longer C5.2
- net at R1.2, R2.2, R3.2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: now also Q1.2 (B)
- net at R10.2, R13.2: now also Q2.3 (C)
- net at C2.2, R9.2, U2.13 (-): now also Q1.3 (C)
- net at R12.1: now also Q1.1 (E), Q2.1 (E)
- net at D1.1 (K), D2.2 (A), R14.2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: now also R16.2
- net at R5.2: now also SW1.1, SW1.2, SW1.6; no longer J1.S
- net at RV4.2, U2.10 (+): no longer R16.2
- new net: J1.S, SW1.3
- new net: SW1.4, SW1.8
- new net: C5.2, SW1.7
Other:
- note added: "Korg MS-20 Clone, with LP/BP/HP switch"
- moved on the sheet: C11, C12, D1, D2, J1, J7, R5, R7

Commit message: Fixed title in Schematic
Other:
- note added: "Korg MS-20 VCF Clone, with LP/BP/HP switch"
- note removed: "Korg MS-20 Clone, with LP/BP/HP switch"
Changed lines of the file:
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@@
     (stroke (width 0) (type solid) (color 0 0 0 0))
   )
-  (text "Korg MS-20 Clone, with LP/BP/HP switch" (at 267.335 176.53 180)
+  (text "Korg MS-20 VCF Clone, with LP/BP/HP switch" (at 273.05 176.53 180)
     (effects (font (size 2.54 2.54)) (justify right bottom))
   )

Commit message: Committed some uncommitted changes
Parts:
- R1, R10, R11, R12, R13, R14, R15, R16, R17, R18, R19, R2, R3, R4, R5, R6, R7, R8, R9: footprint (none) -> Resistor_THT:R_Axial_DIN0207_L6.3mm_D2.5mm_P10.16mm_Horizontal
