File: kicad-projects/VCO-Version-1/VCO-Version-1.kicad_pcb (KiCad board)
At the start: 0 parts

Commit message: Worked more on VCO1 PCB
Parts:
- added C1: 100p, Capacitor_THT:C_Rect_L7.0mm_W3.5mm_P5.00mm, F.Cu at (55.3, 87.7)
- added C10: 47n, Capacitor_THT:C_Rect_L7.0mm_W3.5mm_P5.00mm, B.Cu at (192.0, 143.6)
- added C11: 47p, Capacitor_THT:C_Rect_L7.0mm_W3.5mm_P5.00mm, B.Cu at (237.2, 61.6)
- added C12: 100n, Capacitor_THT:C_Rect_L7.0mm_W3.5mm_P5.00mm, B.Cu at (204.6, 143.6)
- added C13: 47u, Capacitor_THT:CP_Radial_D6.3mm_P2.50mm, B.Cu at (199.0, 150.8)
- added C2: 100n, Capacitor_THT:C_Rect_L7.0mm_W3.5mm_P5.00mm, B.Cu at (174.5, 126.0)
- added C3: 100n, Capacitor_THT:C_Rect_L7.0mm_W3.5mm_P5.00mm, B.Cu at (178.8, 121.0)
- added C4: 100n, Capacitor_THT:C_Rect_L7.0mm_W3.5mm_P5.00mm, B.Cu at (238.8, 92.8)
- added C5: 100n, Capacitor_THT:C_Rect_L7.0mm_W3.5mm_P5.00mm, B.Cu at (241.8, 43.8)
- added C6: 47u, Capacitor_THT:CP_Radial_D6.3mm_P2.50mm, B.Cu at (116.9, 135.6)
- added C7: 47u, Capacitor_THT:CP_Radial_D6.3mm_P2.50mm, B.Cu at (116.8, 127.9)
- added C8: 2n2, Capacitor_THT:C_Rect_L7.0mm_W3.5mm_P5.00mm, B.Cu at (166.1, 132.0)
- added C9: 4n7, Capacitor_THT:C_Rect_L7.0mm_W3.5mm_P5.00mm, B.Cu at (189.4, 123.1)
- added D1: D, Diode_THT:D_DO-35_SOD27_P7.62mm_Horizontal, F.Cu at (55.2, 92.2)
- added D2: D, Diode_THT:D_DO-35_SOD27_P7.62mm_Horizontal, B.Cu at (159.4, 123.2)
- added D3: D, Diode_THT:D_DO-35_SOD27_P7.62mm_Horizontal, B.Cu at (187.4, 126.6)
- added D4: D, Diode_THT:D_DO-35_SOD27_P7.62mm_Horizontal, B.Cu at (251.6, 101.5)
- added D5: D, Diode_THT:D_DO-35_SOD27_P7.62mm_Horizontal, B.Cu at (258.9, 98.2)
- added D6: D, Diode_THT:D_DO-35_SOD27_P7.62mm_Horizontal, B.Cu at (190.0, 134.2)
- added J1: CV, Connector_Audio:Jack_3.5mm_QingPu_WQP-PJ398SM_Vertical_CircularHoles, F.Cu at (37.8, 121.8)
- added J10: C2T, Connector_PinHeader_2.54mm:PinHeader_1x06_P2.54mm_Vertical, B.Cu at (34.0, 80.2)
- added J11: C1B, Connector_PinSocket_2.54mm:PinSocket_1x06_P2.54mm_Vertical, F.Cu at (129.0, 80.2)
- added J12: C2B, Connector_PinSocket_2.54mm:PinSocket_1x06_P2.54mm_Vertical, F.Cu at (87.0, 80.2)
- added J13: Power, Connector_IDC:IDC-Header_2x05_P2.54mm_Vertical, B.Cu at (128.0, 125.4)
- added J2: Exp FM, Connector_Audio:Jack_3.5mm_QingPu_WQP-PJ398SM_Vertical_CircularHoles, F.Cu at (49.2, 121.8)
- added J3: Lin FM, Connector_Audio:Jack_3.5mm_QingPu_WQP-PJ398SM_Vertical_CircularHoles, F.Cu at (60.8, 121.8)
- added J4: Sync, Connector_Audio:Jack_3.5mm_QingPu_WQP-PJ398SM_Vertical_CircularHoles, F.Cu at (37.8, 136.8)
- added J5: CV_PWM, Connector_Audio:Jack_3.5mm_QingPu_WQP-PJ398SM_Vertical_CircularHoles, F.Cu at (72.2, 121.8)
- added J6: Saw, Connector_Audio:Jack_3.5mm_QingPu_WQP-PJ398SM_Vertical_CircularHoles, F.Cu at (49.2, 136.8)
- added J7: Tri, Connector_Audio:Jack_3.5mm_QingPu_WQP-PJ398SM_Vertical_CircularHoles, F.Cu at (60.8, 136.8)
- added J8: Pulse, Connector_Audio:Jack_3.5mm_QingPu_WQP-PJ398SM_Vertical_CircularHoles, F.Cu at (72.2, 137.0)
- added J9: C1T, Connector_PinHeader_2.54mm:PinHeader_1x06_P2.54mm_Vertical, B.Cu at (76.0, 80.2)
- added Q1: NPN, Package_TO_SOT_THT:TO-92_Inline, B.Cu at (156.9, 141.4)
- added Q2: NPN, Package_TO_SOT_THT:TO-92_Inline, B.Cu at (159.5, 137.4)
- added Q3: Q_NPN_CBE, Package_TO_SOT_THT:TO-92_Inline, B.Cu at (189.2, 144.1)
- added R1: 100k, Resistor_THT:R_Axial_DIN0207_L6.3mm_D2.5mm_P7.62mm_Horizontal, F.Cu at (51.0, 64.2)
- added R10: 2M2, Resistor_THT:R_Axial_DIN0207_L6.3mm_D2.5mm_P7.62mm_Horizontal, F.Cu at (55.5, 69.2)
- added R11: 100k, Resistor_THT:R_Axial_DIN0207_L6.3mm_D2.5mm_P7.62mm_Horizontal, B.Cu at (169.6, 144.6)
- added R12: R, Resistor_THT:R_Axial_DIN0207_L6.3mm_D2.5mm_P7.62mm_Horizontal, B.Cu at (153.9, 139.2)
- added R13: 10k, Resistor_THT:R_Axial_DIN0207_L6.3mm_D2.5mm_P7.62mm_Horizontal, B.Cu at (168.7, 142.0)
- added R14: 2k2, Resistor_THT:R_Axial_DIN0207_L6.3mm_D2.5mm_P7.62mm_Horizontal, B.Cu at (162.0, 147.6)
- added R15: R, Resistor_THT:R_Axial_DIN0207_L6.3mm_D2.5mm_P7.62mm_Horizontal, B.Cu at (162.0, 150.7)
- added R16: 100k, Resistor_THT:R_Axial_DIN0207_L6.3mm_D2.5mm_P7.62mm_Horizontal, B.Cu at (153.9, 129.4)
- added R17: 100k, Resistor_THT:R_Axial_DIN0207_L6.3mm_D2.5mm_P7.62mm_Horizontal, B.Cu at (194.1, 150.9)
- added R18: 1M, Resistor_THT:R_Axial_DIN0207_L6.3mm_D2.5mm_P7.62mm_Horizontal, B.Cu at (169.6, 132.2)
- added R19: 47k, Resistor_THT:R_Axial_DIN0207_L6.3mm_D2.5mm_P7.62mm_Horizontal, B.Cu at (244.8, 102.0)
- added R2: 100k, Resistor_THT:R_Axial_DIN0207_L6.3mm_D2.5mm_P7.62mm_Horizontal, F.Cu at (69.4, 85.1)
- added R20: 47k, Resistor_THT:R_Axial_DIN0207_L6.3mm_D2.5mm_P7.62mm_Horizontal, B.Cu at (263.2, 58.4)
- added R21: 100k, Resistor_THT:R_Axial_DIN0207_L6.3mm_D2.5mm_P7.62mm_Horizontal, B.Cu at (194.1, 153.9)
- added R22: 1k8, Resistor_THT:R_Axial_DIN0207_L6.3mm_D2.5mm_P7.62mm_Horizontal, B.Cu at (165.7, 141.9)
- added R23: 1k, Resistor_THT:R_Axial_DIN0207_L6.3mm_D2.5mm_P7.62mm_Horizontal, B.Cu at (162.6, 134.4)
- added R24: 47k, Resistor_THT:R_Axial_DIN0207_L6.3mm_D2.5mm_P7.62mm_Horizontal, B.Cu at (251.3, 82.6)
- added R25: 1k, Resistor_THT:R_Axial_DIN0207_L6.3mm_D2.5mm_P7.62mm_Horizontal, B.Cu at (183.7, 142.4)
- added R26: 470, Resistor_THT:R_Axial_DIN0207_L6.3mm_D2.5mm_P7.62mm_Horizontal, B.Cu at (184.6, 126.6)
- added R27: 100k, Resistor_THT:R_Axial_DIN0207_L6.3mm_D2.5mm_P7.62mm_Horizontal, B.Cu at (263.2, 67.9)
- added R28: 10k, Resistor_THT:R_Axial_DIN0207_L6.3mm_D2.5mm_P7.62mm_Horizontal, B.Cu at (259.6, 83.8)
- added R29: 1M, Resistor_THT:R_Axial_DIN0207_L6.3mm_D2.5mm_P7.62mm_Horizontal, B.Cu at (191.8, 136.8)
- added R3: 100k, Resistor_THT:R_Axial_DIN0207_L6.3mm_D2.5mm_P7.62mm_Horizontal, F.Cu at (51.0, 58.2)
- added R30: 100k, Resistor_THT:R_Axial_DIN0207_L6.3mm_D2.5mm_P7.62mm_Horizontal, B.Cu at (268.8, 83.3)
- added R31: 2k2, Resistor_THT:R_Axial_DIN0207_L6.3mm_D2.5mm_P7.62mm_Horizontal, B.Cu at (184.2, 139.8)
- added R32: 100k, Resistor_THT:R_Axial_DIN0207_L6.3mm_D2.5mm_P7.62mm_Horizontal, B.Cu at (222.6, 86.5)
- added R33: 50k, Resistor_THT:R_Axial_DIN0207_L6.3mm_D2.5mm_P7.62mm_Horizontal, B.Cu at (230.0, 75.2)
- added R34: R, Resistor_THT:R_Axial_DIN0207_L6.3mm_D2.5mm_P7.62mm_Horizontal, B.Cu at (241.7, 67.2)
- added R35: R, Resistor_THT:R_Axial_DIN0207_L6.3mm_D2.5mm_P7.62mm_Horizontal, B.Cu at (232.1, 49.8)
- added R36: 100, Resistor_THT:R_Axial_DIN0207_L6.3mm_D2.5mm_P7.62mm_Horizontal, B.Cu at (194.2, 128.9)
- added R37: 150k, Resistor_THT:R_Axial_DIN0207_L6.3mm_D2.5mm_P7.62mm_Horizontal, B.Cu at (252.4, 58.7)
- added R38: 200k, Resistor_THT:R_Axial_DIN0207_L6.3mm_D2.5mm_P7.62mm_Horizontal, B.Cu at (238.2, 57.5)
- added R39: R, Resistor_THT:R_Axial_DIN0207_L6.3mm_D2.5mm_P7.62mm_Horizontal, B.Cu at (222.8, 48.5)
- added R4: 3M3, Resistor_THT:R_Axial_DIN0207_L6.3mm_D2.5mm_P7.62mm_Horizontal, F.Cu at (69.2, 62.5)
- added R40: 10R, Resistor_THT:R_Axial_DIN0207_L6.3mm_D2.5mm_P7.62mm_Horizontal, B.Cu at (186.5, 147.7)
- added R41: 1k, Resistor_THT:R_Axial_DIN0207_L6.3mm_D2.5mm_P7.62mm_Horizontal, B.Cu at (224.9, 71.9)
- added R5: R, Resistor_THT:R_Axial_DIN0207_L6.3mm_D2.5mm_P7.62mm_Horizontal, F.Cu at (72.9, 104.7)
- added R6: R, Resistor_THT:R_Axial_DIN0207_L6.3mm_D2.5mm_P7.62mm_Horizontal, F.Cu at (43.5, 104.7)
- added R7: R, Resistor_THT:R_Axial_DIN0207_L6.3mm_D2.5mm_P7.62mm_Horizontal, F.Cu at (48.6, 85.1)
- added R8: R, Resistor_THT:R_Axial_DIN0207_L6.3mm_D2.5mm_P7.62mm_Horizontal, F.Cu at (62.9, 104.7)
- added R9: 0R, Resistor_THT:R_Axial_DIN0207_L6.3mm_D2.5mm_P7.62mm_Horizontal, F.Cu at (58.6, 61.2)
- added REF**: MountingHole_3.2mm_M3_ISO14580_Pad, MountingHole:MountingHole_3.2mm_M3_ISO14580_Pad, F.Cu at (55.0, 138.0)
- added REF**: MountingHole_3.2mm_M3_ISO14580_Pad, MountingHole:MountingHole_3.2mm_M3_ISO14580_Pad, F.Cu at (108.0, 138.0)
- added REF**: MountingHole_3.2mm_M3_ISO14580_Pad, MountingHole:MountingHole_3.2mm_M3_ISO14580_Pad, F.Cu at (108.0, 45.0)
- added REF**: MountingHole_3.2mm_M3_ISO14580_Pad, MountingHole:MountingHole_3.2mm_M3_ISO14580_Pad, F.Cu at (55.0, 45.0)
- added RV1: FM Level, Potentiometer_THT:Potentiometer_Alpha_RD901F-40-00D_Single_Vertical, F.Cu at (64.5, 79.7)
- added RV10: 50k, Potentiometer_THT:Potentiometer_Bourns_3296W_Vertical, B.Cu at (158.2, 127.0)
- added RV11: 50k, Potentiometer_THT:Potentiometer_Bourns_3296W_Vertical, B.Cu at (254.2, 46.0)
- added RV2: Coarse Freq, Potentiometer_THT:Potentiometer_Alpha_RD901F-40-00D_Single_Vertical, F.Cu at (42.6, 53.6)
- added RV3: Fine Freq, Potentiometer_THT:Potentiometer_Alpha_RD901F-40-00D_Single_Vertical, F.Cu at (66.8, 58.3)
- added RV4: Lin FM Level, Potentiometer_THT:Potentiometer_Alpha_RD901F-40-00D_Single_Vertical, F.Cu at (41.0, 79.7)
- added RV5: PWM Level, Potentiometer_THT:Potentiometer_Alpha_RD901F-40-00D_Single_Vertical, F.Cu at (64.5, 101.1)
- added RV6: PWM Offset, Potentiometer_THT:Potentiometer_Alpha_RD901F-40-00D_Single_Vertical, F.Cu at (41.0, 101.1)
- added RV7: 50k, Potentiometer_THT:Potentiometer_Bourns_3296W_Vertical, B.Cu at (178.3, 149.4)
- added RV8: 50k, Potentiometer_THT:Potentiometer_Bourns_3296W_Vertical, B.Cu at (158.2, 151.8)
- added RV9: 50k, Potentiometer_THT:Potentiometer_Bourns_3296W_Vertical, B.Cu at (238.5, 100.4)
- added TH1: 10k, Resistor_THT:R_Axial_DIN0207_L6.3mm_D2.5mm_P2.54mm_Vertical, B.Cu at (162.4, 139.4)
- added U1: TL074, Package_DIP:DIP-14_W7.62mm_Socket, B.Cu at (172.9, 144.5)
- added U2: TL074, Package_DIP:DIP-14_W7.62mm_Socket, B.Cu at (234.3, 85.7)
- added U3: ICM7555xP, Package_DIP:DIP-8_W7.62mm, B.Cu at (201.8, 132.2)
Other:
- board outline added: 100 x 100 mm
- copper layers 0 -> 2
