File: kicad-projects/VCO-Version-1/VCO-Version-1.kicad_pcb (KiCad board)
At the start: 2 copper layers, 100 x 100 mm, 95 parts, among them J1 CV, J10 C2T, J11 C1B, J12 C2B, J13 Power, J2 Exp FM, J3 Lin FM, J4 Sync, J5 CV_PWM, J6 Saw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

Commit message: More work on layout on PCB
Parts:
- moved R20 127.6 mm to (167.4, 142.7)
- moved R27 123.3 mm to (163.2, 140.0), turned to 90 degrees
- moved C5 114.3 mm to (169.8, 132.6), turned to -90 degrees
- moved R37 112.0 mm to (178.4, 142.7), turned to 0 degrees
- moved R30 111.0 mm to (173.4, 140.0)
- moved RV11 107.2 mm to (185.3, 128.1), turned to -90 degrees
- moved R35 103.0 mm to (182.4, 140.0), turned to 90 degrees
- moved D5 101.0 mm to (160.0, 118.5), turned to 90 degrees
- moved R28 100.5 mm to (176.4, 140.0)
- moved R39 98.9 mm to (185.4, 140.0), turned to 90 degrees
- moved R24 98.6 mm to (166.2, 132.4), turned to -90 degrees
- moved RV6 91.5 mm to (131.9, 90.4)
- moved R34 90.1 mm to (179.4, 132.4), turned to -90 degrees
- moved R19 89.9 mm to (160.2, 132.4), turned to -90 degrees
- moved D4 89.5 mm to (162.5, 110.9), turned to -90 degrees
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
Commit message: Added completed PCB layout which will likely be ordered.
Parts:
- added REF**: MouseBites_5x2mm+0.5mm, MouseBites:MouseBites_5x2mm+0.5mm, F.Cu at (146.9, 125.7)
- added REF**: MouseBites_5x2mm+0.5mm, MouseBites:MouseBites_5x2mm+0.5mm, F.Cu at (146.9, 75.2)
- moved C11 45.2 mm to (152.3, 145.0), turned to 90 degrees
- moved R38 42.3 mm to (159.5, 147.5), turned to 90 degrees
- moved D4 40.8 mm to (180.7, 147.4), turned to 90 degrees
- moved R39 40.8 mm to (152.8, 115.5), turned to -90 degrees
- moved R37 36.7 mm to (159.9, 111.0), turned to 180 degrees
- moved R35 36.0 mm to (156.1, 115.4), turned to -90 degrees
- moved R6 34.1 mm to (124.3, 84.0), turned to -90 degrees
- moved R20 31.9 mm to (174.6, 111.6), turned to 0 degrees
- moved D5 31.7 mm to (183.5, 139.8), turned to -90 degrees
- moved RV11 31.3 mm to (154.0, 129.0), turned to 90 degrees
- moved R41 30.4 mm to (156.2, 139.8), turned to -90 degrees
- moved R27 28.9 mm to (178.5, 115.4), turned to -90 degrees
- moved R28 26.7 mm to (166.0, 115.4), turned to -90 degrees
- moved R32 24.6 mm to (177.6, 139.8), turned to -90 degrees
- moved R33 24.5 mm to (162.8, 139.8), turned to -90 degrees
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Connections:
- D1 pad 2: GND -> GNDA
- J10 pad 1: GNDA -> /P_FMlin
- J10 pad 3: /P_HFtrim -> /P_OSaw
- J10 pad 4: /P_FMlin -> /P_OPulse
- J10 pad 5: /P_Sync -> GNDA
- J10 pad 6: /P_PWMoffs -> /P_OTri
- J11 pad 1: +12V -> /HFtrim
- J11 pad 2: /OSaw -> /Sync
- J11 pad 3: /OTri -> /PWMoffs
- J11 pad 4: /OPulse -> +12V
- J11 pad 5: -12V -> GND
- J11 pad 6: GND -> -12V
- J12 pad 1: GND -> /FMlin
- J12 pad 3: /HFtrim -> /OSaw
- J12 pad 4: /FMlin -> /OPulse
- J12 pad 5: /Sync -> GND
- J12 pad 6: /PWMoffs -> /OTri
- J4 pad S: GND -> GNDA
- J5 pad S: GND -> GNDA
- J6 pad S: Net-(J6-PadS) -> GNDA
- J7 pad S: Net-(J6-PadS) -> GNDA
- J8 pad S: Net-(J6-PadS) -> GNDA
- J9 pad 1: +12VA -> /P_HFtrim
- J9 pad 2: /P_OSaw -> /P_Sync
- J9 pad 3: /P_OTri -> /P_PWMoffs
- J9 pad 4: /P_OPulse -> +12VA
- J9 pad 5: -12VA -> GNDA
- J9 pad 6: GNDA -> -12VA
- R8 pad 2: GND -> GNDA
- REF** pad 1: (no net) -> GNDA (x2)
- REF** pad 1: (no net) -> GND (x2)
- RV5 pad 3: GND -> GNDA
Routing:
- net +12V: track 0.00 -> 177.2 mm, vias 0 -> 1
- net -12V: track 0.00 -> 106.6 mm
- net +12VA: track 0.00 -> 66.8 mm
- net /P_OPulse: track 0.00 -> 59.3 mm
- net /WSaw: track 0.00 -> 57.7 mm
- net /CVmix: track 0.00 -> 57.0 mm
- net Net-(J1-PadT): track 0.00 -> 53.0 mm
- net /OTri: track 0.00 -> 50.6 mm
- net /PWMoffs: track 0.00 -> 48.7 mm
- net Net-(C11-Pad1): track 0.00 -> 48.5 mm
- net /P_OSaw: track 0.00 -> 47.4 mm
- net /P_PWMoffs: track 0.00 -> 47.3 mm
- net /WRoot: track 0.00 -> 44.3 mm
- net /P_OTri: track 0.00 -> 43.2 mm
- net Net-(C1-Pad1): track 0.00 -> 41.5 mm
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- added copper zone on B.Cu, net GND
- added copper zone on F.Cu, net GND
- added copper zone on B.Cu, net GNDA
- added copper zone on F.Cu, net GNDA
Other:
- board size 100 x 100 mm -> 96 x 100 mm
