File: kicad-projects/MS20-Plus-VCF-v2/MS20-Plus-VCF-v2.kicad_pcb (KiCad board)
At the start: 2 copper layers, 87 x 100 mm, 78 parts, among them J1 CV1, J10 PanelC2, J11 BackC2, J2 CV2, J3 CV3, J4 Out, J5 HP_In, J6 LP_In, J7 EURPower, J8 PanelC1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

Commit message: Added gerbers and final updates before ordering
Parts:
- added REF**: MouseBites_5x2mm+0.5mm, Mousebites:MouseBites_5x2mm+0.5mm, F.Cu at (77.5, 70.7)
- added REF**: MouseBites_5x2mm+0.5mm, Mousebites:MouseBites_5x2mm+0.5mm, F.Cu at (77.5, 113.2)
- moved C1 9.00 mm to (94.7, 89.3)
- moved C10 9.00 mm to (93.1, 143.4)
- moved C2 9.00 mm to (85.5, 73.2)
- moved C3 9.00 mm to (82.2, 90.0)
- moved C4 9.00 mm to (110.6, 91.0)
- moved C5 9.00 mm to (113.2, 55.4)
- moved C6 9.00 mm to (94.7, 84.5)
- moved C7 9.00 mm to (102.1, 65.4)
- moved C8 9.00 mm to (84.8, 143.3)
- moved C9 9.00 mm to (107.1, 132.2)
- moved J11 9.00 mm to (114.8, 121.5)
- moved J7 9.00 mm to (113.2, 68.0)
- moved J9 9.00 mm to (80.3, 121.5)
- moved Q1 9.00 mm to (99.4, 107.2)
- moved Q2 9.00 mm to (95.4, 104.6)
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Routing:
- net -12VA: track 83.7 -> 82.4 mm
- net /SC_LpG2_P: track 76.8 -> 77.7 mm
- net /FPole2: track 45.3 -> 46.1 mm
- net /HP_In: track 13.1 -> 13.8 mm
- net +12V: track 126.3 -> 126.9 mm
- net Net-(C8-Pad2): track 54.4 -> 54.9 mm
- net GND: vias 84 -> 87
Other:
- board size 87 x 100 mm -> 78 x 100.1 mm
